File: Hardware/KrzempolDriver.kicad_sch (KiCad schematic)
At the start: 42 parts, among them J1 24V, U1 RT6285, U2 RT6285, U3 RT6285

Commit message: driver and output
Parts:
- removed A1: Arduino_Nano_RP2040_Connect, Module:Arduino_Nano, symbol MCU_Module:Arduino_Nano_RP2040_Connect
- added D4: MBR120VLSFT, symbol Device:D_Schottky
- added JP5: Jumper_2_Open, symbol Jumper:Jumper_2_Open
- added U4: RASPBERRY-PI-PICO, Module_RaspberryPi_Pico:RaspberryPi_Pico_Common, symbol krzempol:RASPBERRY-PI-PICO
Connections:
- net +3.3V_PI: now also U4.36 (3V3)
- net +5V: now also D4.2 (A)
- net GND: now also JP5.1 (A), U4.13 (GND), U4.18 (GND), U4.23 (GND), U4.28 (GND), U4.3 (GND), U4.33 (AGND), U4.38 (GND), U4.8 (GND)
- new net: JP5.2 (B), U4.37 (3V3_EN)
- new net: D4.1 (K), U4.39 (VSYS)
- new net DRIVER/PH1: U4.27 (GPIO21)
- new net DRIVER/PH2: U4.25 (GPIO19)
- new net DRIVER/PH3: U4.22 (GPIO17)
- new net DRIVER/ZC1: U4.26 (GPIO20)
- new net DRIVER/ZC2: U4.24 (GPIO18)
- new net DRIVER/ZC3: U4.21 (GPIO16)
- new net OUTPUT/INPUT1: U4.1 (GPIO0)
- new net OUTPUT/INPUT2: U4.4 (GPIO2)
- new net OUTPUT/INPUT3: U4.6 (GPIO4)
- new net OUTPUT/INPUT4: U4.9 (GPIO6)
- no-connect marks 0 -> 3
Other:
- sheet driver renamed DRIVER
- added sheet OUTPUT (output.kicad_sch)
- sheet DRIVER ports: added PH1, PH2, PH3, ZC1, ZC2, ZC3; removed none
- note added: "OPTIONAL"
- moved on the sheet: C1, C14, C15, C16, C17, C18, C19, C20, C21, D3, J1, JP3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

Commit message: minor fixes
Parts:
- added C32, C33: 100n, symbol Device:C
- added J13, J14: MAX31865, symbol Connector_Generic:Conn_01x08
- added J15, J16: Conn_01x03, symbol Connector_Generic:Conn_01x03
Connections:
- net +3.3V: now also C32.2, C33.2, J13.3 (Pin_3), J14.3 (Pin_3)
- net GND: now also C32.1, C33.1, J13.2 (Pin_2), J14.2 (Pin_2)
- net SDO1: now reaches U4.10 (GPIO7)
- net SDO1: now also J13.5 (Pin_5)
- net CLK1: now reaches U4.11 (GPIO8)
- net CLK1: now also J13.4 (Pin_4)
- net RDY2: now reaches U4.12 (GPIO9)
- net RDY2: now also J14.8 (Pin_8)
- net CS2: now reaches U4.14 (GPIO10)
- net CS2: now also J14.7 (Pin_7)
- net SDI2: now reaches U4.15 (GPIO11)
- net SDI2: now also J14.6 (Pin_6)
- net SDO2: now reaches U4.16 (GPIO12)
- net SDO2: now also J14.5 (Pin_5)
- net at U4.17 (GPIO13): now also J15.3 (Pin_3)
- net at U4.19 (GPIO14): now also J15.2 (Pin_2)
- net RDY1: now reaches U4.2 (GPIO1)
- net RDY1: now also J13.8 (Pin_8)
- net at U4.20 (GPIO15): now also J15.1 (Pin_1)
- net CLK2: now reaches U4.29 (GPIO22)
- net CLK2: now also J14.4 (Pin_4)
- net at U4.31 (GPIO26_ADC0): now also J16.1 (Pin_1)
- net at U4.32 (GPIO27_ADC1): now also J16.2 (Pin_2)
- net at U4.34 (GPIO28_ADC2): now also J16.3 (Pin_3)
- net CS1: now reaches U4.5 (GPIO3)
- net CS1: now also J13.7 (Pin_7)
- net SDI1: now reaches U4.7 (GPIO5)
- net SDI1: now also J13.6 (Pin_6)
- no-connect marks 3 -> 5
Other:
- company: (none) -> MOS
- title: (none) -> Krzempol furnace
- moved on the sheet: C20, D4, JP5, U4
