File: Hardware/driver.kicad_sch (KiCad schematic)
At the start: 0 parts

Commit message: driver and output
Parts:
- added C26, C27, C28: 100n 400v, symbol Device:C
- added C29, C30, C31: 10u 25V, symbol Device:C_Polarized
- added D10, D11, D13: GREEN, symbol Device:LED
- added D12, D14, D9: BTA330, symbol Device:Q_Triac
- added D15, D17, D19: D_Bridge_+A-A, symbol Device:D_Bridge_+A-A
- added D16, D18, D20: D, symbol Device:D
- added HS1, HS2, HS3: Heatsink_Pad_2Pin, symbol Mechanical:Heatsink_Pad_2Pin
- added J10, J11, J12: Heater, symbol Connector:Screw_Terminal_01x02
- added Q1, Q2, Q3: BSS123, Package_TO_SOT_SMD:SOT-23, symbol Transistor_FET:BSS123
- added Q4, Q5, Q6: MMBT3904, Package_TO_SOT_SMD:SOT-23, symbol Transistor_BJT:MMBT3904
- added R19, R27, R32: 680 2W, symbol Device:R
- added R20, R28, R33: 39 2W, symbol Device:R
- added R21, R26, R31: 220, symbol Device:R
- added R22, R23, R24, R25, R29, R30: 100, symbol Device:R
- added R34, R35, R39, R40, R44, R45: 220k, symbol Device:R
- added R36, R37, R41, R42, R46, R47: 22k, symbol Device:R
- added R38, R43, R48: 10k, symbol Device:R
- added U10, U11, U9: MOC3021M, symbol Relay_SolidState:MOC3021M
- added U12, U13, U14: 4N25, Package_DIP:DIP-6_W7.62mm, symbol Isolator:4N25
Connections:
- new net: D15.3 (-), D16.1 (K), Q4.1 (B), R36.1
- new net: C29.1, D15.1 (+), R36.2, R37.2
- new net: D19.4, R44.2
- new net: C27.1, D12.A1, J11.1 (Pin_1)
- new net: C27.2, R28.1
- new net: R26.2, U10.1
- new net: D11.1 (K), Q2.3 (D), U10.2
- new net: D12.G, U10.4
- new net: R27.1, U10.6
- new net: C28.1, D14.A1, J12.1 (Pin_1)
- new net: D14.G, U11.4
- new net: D13.1 (K), Q3.3 (D), U11.2
- new net: C28.2, R33.1
- new net: R32.1, U11.6
- new net: D10.1 (K), Q1.3 (D), U9.2
- new net: D10.2 (A), R22.1
- new net: R47.1, U14.1
- new net: C31.1, D19.1 (+), R46.2, R47.2
- new net: R19.1, U9.6
- new net: R31.2, U11.1
- new net: D17.4, R39.2
- new net: D15.2, R35.2
- new net: D15.4, R34.2
- new net: C26.2, R20.1
- new net: C26.1, D9.A1, J10.1 (Pin_1)
- new net: D17.2, R40.2
- new net: R42.1, U13.1
- new net: Q5.3 (C), U13.2
- new net: D19.3 (-), D20.1 (K), Q6.1 (B), R46.1
- new net: C31.2, D20.2 (A), Q6.2 (E)
- new net: D11.2 (A), R24.1
- new net: C30.1, D17.1 (+), R41.2, R42.2
- new net: D17.3 (-), D18.1 (K), Q5.1 (B), R41.1
- new net: C30.2, D18.2 (A), Q5.2 (E)
- new net: C29.2, D16.2 (A), Q4.2 (E)
- new net: Q6.3 (C), U14.2
- new net: D13.2 (A), R29.1
- new net: Q4.3 (C), U12.2
- new net: D19.2, R45.2
- new net: R21.2, U9.1
- new net: D9.G, U9.4
- new net: R37.1, U12.1
- new net +3.3V: R21.1, R22.2, R24.2, R26.1, R29.2, R31.1, R38.2, R43.2, R48.2
- new net GND: Q1.2 (S), Q2.2 (S), Q3.2 (S), R23.1, R25.1, R30.1, U12.4, U13.4, U14.4
- new net NEUT: J10.2 (Pin_2), J11.2 (Pin_2), J12.2 (Pin_2), R35.1, R40.1, R45.1
- new net PH1: Q1.1 (G), R23.2
- new net PH2: Q2.1 (G), R25.2
- new net PH3: Q3.1 (G), R30.2
- new net PHASE1: D9.A2, R19.2, R20.2, R34.1
- new net PHASE2: D12.A2, R27.2, R28.2, R39.1
- new net PHASE3: D14.A2, R32.2, R33.2, R44.1
- new net ZC1: R38.1, U12.5
- new net ZC2: R43.1, U13.5
- new net ZC3: R48.1, U14.5
- no-connect marks 0 -> 9
Other:
- note added: "OPTIONAL"

Commit message: minor fixes
Other:
- company: (none) -> MOS
- title: (none) -> Krzempol furnace
Changed lines of the file:
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@@
 	(generator_version "8.0")
 	(paper "A4")
+	(title_block
+		(title "Krzempol furnace")
+		(date "2025-02-18")
+		(rev "1.0")
+		(company "MOS")
+	)
 	(junction
 		(at 210.82 99.06)
