File: Hardware/output.kicad_sch (KiCad schematic)
At the start: 36 parts, among them J2 OUT 1, J3 Conn_02x04_Odd_Even, J4 Conn_02x04_Odd_Even, J5 OUT 1, J6 Conn_02x04_Odd_Even, J7 OUT 1, J8 Conn_02x04_Odd_Even, J9 OUT 1, U5 BTF3050, U6 BTF3050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

Commit message: minor fixes
Other:
- company: (none) -> MOS
- title: (none) -> Krzempol furnace
Changed lines of the file:
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@@
 	(generator_version "8.0")
 	(paper "A4")
+	(title_block
+		(title "Krzempol furnace")
+		(date "2025-02-18")
+		(rev "1.0")
+		(company "MOS")
+	)
 	(junction
 		(at 72.39 137.16)
